File: hardware/ospi_v143+.brd (EAGLE design)
At the start: 83.8 x 63.5 mm, 37 parts, among them J0 ACIN, T1 MAC97, T2 MAC97, T3 MAC97, T4 MAC97, T5 MAC97, T6 MAC97, T7 MAC97, T8 MAC97

Commit message: update
Parts:
- removed F2: (no value), adafruit:1812
- removed J0: ACIN, SparkFun:SCREWTERMINAL-4MM-2-X
- added ACIN: (no value), SparkFun:SCREWTERMINAL-5MM-2-X
- added R10: 3k, resistor:M0805
- added R9: 1k, resistor:M0805
- LM2596-ADJ: value (none) -> LM2596-ADJ
- moved D3 5.08 mm to (11.1, 46.5)
- moved RZ 5.08 mm to (4.60, 46.5)
- moved LED 5.08 mm to (9.95, 53.4)
- moved RLED 5.08 mm to (3.30, 53.3)
- moved C0 2.55 mm to (17.9, 48.3), turned to 90 degrees
- renumbered AP1501 to LM2596-ADJ
Connections:
- removed net VIN_PRE: C0.1, C2.+, F2.1, L1.2, LM2596-ADJ.4
- new net N$4: LM2596-ADJ.4, R10.2, R9.2
- net 24VAC: now also ACIN.2; no longer J0.2
- net GND: now also ACIN.1, R9.1; no longer J0.1
- net VIN: now also C0.1, C2.+, L1.2, R10.1; no longer F2.2
Routing:
- net VIN_PRE: track 35.0 -> 0.00 mm
- net VIN: track 64.0 -> 87.0 mm
- net N$4: track 0.00 -> 16.8 mm
- net GND: track 4.61 -> 3.37 mm
- net 24VAC: track 38.2 -> 37.2 mm
