File: hardware/ospi_v143+.sch (EAGLE design)
At the start: 37 parts, among them J0 ACIN, T1 MAC97, T2 MAC97, T3 MAC97, T4 MAC97, T5 MAC97, T6 MAC97, T7 MAC97, T8 MAC97

Commit message: update
Parts:
- removed F2: (no value), adafruit:PTCFUSE-1812
- removed J0: ACIN, SparkFun:M024MM-X
- added ACIN: (no value), SparkFun:M025MM-X
- added R10: 3k, resistor:R-EU_M0805
- added R9: 1k, resistor:R-EU_M0805
- LM2596-ADJ: value LM2596S -> LM2596-ADJ
- renumbered AP1501 to LM2596-ADJ
Connections:
- removed net VIN_PRE: C0.1, C2.+, F2.1, L1.2, LM2596-ADJ.FB
- new net N$4: LM2596-ADJ.FB, R10.2, R9.2
- net 24VAC: now also ACIN.2; no longer J0.2
- net GND: now also ACIN.1, R9.1; no longer J0.1
- net VIN: now also C0.1, C2.+, L1.2, R10.1; no longer F2.2
Other:
- moved on the sheet: C0, C2, D3, LED, RLED, RZ
