File: hardware/SprinklerBoard-8p.brd (EAGLE design)
At the start: 45.7 x 53.3 mm, 19 parts, among them IC1 ULN2003AD

Commit message: HW update
Parts:
- moved ACIN 1.22 mm to (42.7, 43.7)
Routing:
- net D5: track 21.4 -> 19.0 mm
- net D4: track 20.0 -> 17.7 mm
- net 24VAC: track 11.4 -> 12.6 mm
- net D1: track 14.6 -> 13.4 mm
- net COM: track 91.0 -> 90.3 mm
